Commit message: Add keyboard controller

File: delicar_bringup/description/ros2_control/gazebo_controllers.xacro (robot description, xacro)
@@ -24,21 +24,21 @@
             <fdir1>1 0 0</fdir1>
         </gazebo> -->
-        <gazebo reference="body_link">
+        <gazebo reference="${prefix}chassis_link">
             <mu1>0.0001</mu1>
             <mu2>0.0001</mu2>
         </gazebo>
-        <gazebo reference="front_right_wheel_link">
+        <gazebo reference="${prefix}front_right_wheel_link">
             <mu1>100.0</mu1>
             <mu2>100.0</mu2>
         </gazebo>
-        <gazebo reference="front_left_wheel_link">
+        <gazebo reference="${prefix}front_left_wheel_link">
             <mu1>100.0</mu1>
             <mu2>100.0</mu2>
         </gazebo>
-        <gazebo reference="rear_right_wheel_link">
+        <gazebo reference="${prefix}rear_right_wheel_link">
             <mu1>100.0</mu1>
             <mu2>100.0</mu2>
         </gazebo>
-        <gazebo reference="rear_left_wheel_link">
+        <gazebo reference="${prefix}rear_left_wheel_link">
             <mu1>100.0</mu1>
             <mu2>100.0</mu2>
@@ -51,4 +51,7 @@
             <mu1>1.0</mu1>
             <mu2>1.0</mu2>
+        </gazebo>
+        <gazebo reference="${prefix}chassis_link">
+            <material>Gazebo/Red</material>
         </gazebo>
         <!-- Gazebo Control -->
@@ -78,6 +81,6 @@
                 <param name="max">${max_velocity}</param>
             </command_interface>
-            <state_interface name="position"/>
-            <state_interface name="velocity"/>
+            <state_interface name="velocity" />
+            <state_interface name="position" />
         </joint>
         <joint name="rear_right_wheel_joint">
@@ -86,6 +89,6 @@
                 <param name="max">${max_velocity}</param>
             </command_interface>
-            <state_interface name="position"/>
-            <state_interface name="velocity"/>
+            <state_interface name="velocity" />
+            <state_interface name="position" />
         </joint>
         </ros2_control>

File: delicar_bringup/description/urdf/delicar_description.urdf.xacro (robot description, xacro)
@@ -28,5 +28,5 @@
           <box size="${base_length} ${base_width} ${base_height}"/>
         </geometry>
-        <material name="orange"/>
+        <material name="red"/>
       </visual>
       <inertial>
@@ -53,11 +53,11 @@
     <link name="${prefix}rear_right_wheel">
       <collision>
-        <origin xyz="0 0 0" rpy="${PI/2} 0 ${PI/2}"/>
-        <geometry>
-          <cylinder length="${wheel_len}" radius="${wheel_radius}"/>
-        </geometry>
-      </collision>
-      <visual>
-        <origin xyz="0 0 0" rpy="${PI/2} 0 ${PI/2}"/>
+        <origin xyz="0 0 0" rpy="0 0 0"/>
+        <geometry>
+          <cylinder length="${wheel_len}" radius="${wheel_radius}"/>
+        </geometry>
+      </collision>
+      <visual>
+        <origin xyz="0 0 0" rpy="0 0 0"/>
         <geometry>
           <cylinder length="${wheel_len}" radius="${wheel_radius}"/>
@@ -66,5 +66,5 @@
       </visual>
       <inertial>
-        <origin xyz="0 0 0" rpy="${PI/2} 0 ${PI/2}"/>
+        <origin xyz="0 0 0" rpy="0 0 0"/>
         <mass value="${wheel_mass}"/>
         <inertia
@@ -80,6 +80,6 @@
       <parent link="${prefix}chassis_link"/>
       <child link="${prefix}rear_right_wheel"/>
-      <origin xyz="-${wheelbase/2} ${base_width/2} -${base_height/2}" rpy="0 0 ${PI/2}"/>
-      <axis xyz="1 0 0"/>
+      <origin xyz="-${wheelbase/2} ${base_width/2} -${base_height/2}" rpy="-${PI/2} 0 0"/>
+      <axis xyz="0 0 1"/>
       <limit effort="10.0" velocity="50.0"/>
       <dynamics damping="0.2"/>
@@ -88,5 +88,5 @@
     <link name="${prefix}rear_left_wheel">
         <collision>
-          <origin xyz="0 0 0" rpy="${PI/2} 0 ${PI/2}"/>
+          <origin xyz="0 0 0" rpy="0 0 0"/>
           <geometry>
             <cylinder length="${wheel_len}" radius="${wheel_radius}"/>
@@ -94,5 +94,5 @@
         </collision>
         <visual>
-          <origin xyz="0 0 0" rpy="${PI/2} 0 ${PI/2}"/>
+          <origin xyz="0 0 0" rpy="0 0 0"/>
           <geometry>
             <cylinder length="${wheel_len}" radius="${wheel_radius}"/>
@@ -101,5 +101,5 @@
         </visual>
         <inertial>
-          <origin xyz="0 0 0" rpy="${PI/2} 0 ${PI/2}"/>
+          <origin xyz="0 0 0" rpy="0 0 0"/>
           <mass value="${wheel_mass}"/>
           <inertia
@@ -115,6 +115,6 @@
       <parent link="${prefix}chassis_link" />
       <child link="${prefix}rear_left_wheel" />
-      <origin xyz="-${wheelbase/2} -${base_width/2} -${base_height/2}" rpy="0 0 ${PI/2}"/>
-      <axis xyz="1 0 0"/>
+      <origin xyz="-${wheelbase/2} -${base_width/2} -${base_height/2}" rpy="-${PI/2} 0 0"/>
+      <axis xyz="0 0 1"/>
       <limit effort="10.0" velocity="50.0"/>
       <dynamics damping="0.2"/>
@@ -152,6 +152,6 @@
       <parent link="${prefix}chassis_link"/>
       <child link="${prefix}front_right_steering_link"/>
-      <origin xyz="${wheelbase/2} ${base_width/2} -${base_height/2}" rpy="0 0 0"/>
-      <axis xyz="0 0 1"/>
+      <origin xyz="${wheelbase/2} ${base_width/2} -${base_height/2}" rpy="${PI/2} 0 0"/>
+      <axis xyz="0 1 0"/>
       <limit lower="-${PI/4}" upper="${PI/4}" effort="50.0" velocity="1.0"/>
       <dynamics damping="0.1"/>
@@ -188,6 +188,6 @@
       <parent link="${prefix}chassis_link"/>
       <child link="${prefix}front_left_steering_link"/>
-      <origin xyz="${wheelbase/2} -${base_width/2} -${base_height/2}" rpy="0 0 0"/>
-      <axis xyz="0 0 1"/>
+      <origin xyz="${wheelbase/2} -${base_width/2} -${base_height/2}" rpy="${PI/2} 0 0"/>
+      <axis xyz="0 1 0"/>
       <limit lower="-${PI/4}" upper="${PI/4}" effort="50.0" velocity="1.0"/>
       <dynamics damping="0.1"/>
@@ -197,11 +197,11 @@
     <link name="${prefix}front_right_wheel">
       <collision>
-        <origin xyz="0 0 0" rpy="${PI/2} 0 ${PI/2}"/>
-        <geometry>
-          <cylinder length="${wheel_len}" radius="${wheel_radius}"/>
-        </geometry>
-      </collision>
-      <visual>
-        <origin xyz="0 0 0" rpy="${PI/2} 0 ${PI/2}"/>
+        <origin xyz="0 0 0" rpy="0 0 0"/>
+        <geometry>
+          <cylinder length="${wheel_len}" radius="${wheel_radius}"/>
+        </geometry>
+      </collision>
+      <visual>
+        <origin xyz="0 0 0" rpy="0 0 0"/>
         <geometry>
           <cylinder length="${wheel_len}" radius="${wheel_radius}"/>
@@ -210,5 +210,5 @@
       </visual>
       <inertial>
-        <origin xyz="0 0 0" rpy="${PI/2} 0 ${PI/2}"/>
+        <origin xyz="0 0 0" rpy="0 0 0"/>
         <mass value="${wheel_mass}"/>
         <inertia
@@ -224,6 +224,6 @@
       <parent link="${prefix}front_right_steering_link" />
       <child link="${prefix}front_right_wheel" />
-      <origin xyz="0 0 0" rpy="0 0 ${PI/2}"/>
-      <axis xyz="1 0 0"/>
+      <origin xyz="0 0 0" rpy="0 0 0"/>
+      <axis xyz="0 0 1"/>
       <limit effort="10.0" velocity="50.0"/>
       <dynamics damping="0.2"/>
@@ -232,11 +232,11 @@
     <link name="${prefix}front_left_wheel">
       <collision>
-        <origin xyz="0 0 0" rpy="${PI/2} 0 ${PI/2}"/>
-        <geometry>
-          <cylinder length="${wheel_len}" radius="${wheel_radius}"/>
-        </geometry>
-      </collision>
-      <visual>
-        <origin xyz="0 0 0" rpy="${PI/2} 0 ${PI/2}"/>
+        <origin xyz="0 0 0" rpy="0 0 0"/>
+        <geometry>
+          <cylinder length="${wheel_len}" radius="${wheel_radius}"/>
+        </geometry>
+      </collision>
+      <visual>
+        <origin xyz="0 0 0" rpy="0 0 0"/>
         <geometry>
           <cylinder length="${wheel_len}" radius="${wheel_radius}"/>
@@ -245,5 +245,5 @@
       </visual>
       <inertial>
-        <origin xyz="0 0 0" rpy="${PI/2} 0 ${PI/2}"/>
+        <origin xyz="0 0 0" rpy="0 0 0"/>
         <mass value="${wheel_mass}"/>
         <inertia
@@ -259,6 +259,6 @@
       <parent link="${prefix}front_left_steering_link" />
       <child link="${prefix}front_left_wheel" />
-      <origin xyz="0 0 0" rpy="0 0 ${PI/2}"/>
-      <axis xyz="1 0 0"/>
+      <origin xyz="0 0 0" rpy="0 0 0"/>
+      <axis xyz="0 0 1"/>
       <limit effort="10.0" velocity="50.0"/>
       <dynamics damping="0.2"/>
