Commit message: Modified urdf to fix strange movement in Gazebo

File: delicar_bringup/description/ros2_control/gazebo_controllers.xacro (robot description, xacro)
@@ -3,101 +3,39 @@
     <xacro:property name="PI" value="3.1415926535897931"/>
     <!-- Arguments -->
-    <xacro:arg name="max_steering_angle" default="0.872665" />
-    <xacro:arg name="max_steering_angular_velocity" default="${PI/4}" />
-    <xacro:arg name="max_steering_effort" default="10.0" />
+    <xacro:arg name="max_steering_angle" default="1.04" />
     <xacro:arg name="max_velocity" default="5.0" />
-    <xacro:arg name="max_effort" default="100.0" />
     <!-- Vehicle Properties -->
     <xacro:property name="max_steering_angle" value="$(arg max_steering_angle)"/>
-    <xacro:property name="max_steering_angular_velocity" value="$(arg max_steering_angular_velocity)"/>
-    <xacro:property name="max_steering_effort" value="$(arg max_steering_effort)"/>
     <xacro:property name="max_velocity" value="$(arg max_velocity)"/>
-    <xacro:property name="max_effort" value="$(arg max_effort)"/>
     <xacro:macro name="gazebo_ros2_control" params="name prefix">
-        <!-- Gazebo Parameters -->
-        <!-- <gazebo reference="${prefix}front_right_wheel_link">
-            <mu1>1.0</mu1>
-            <mu2>1.0</mu2>
-            <kp>100000000.0</kp>
-            <kd>10000.0</kd>
-            <minDepth>0.001</minDepth>
-            <fdir1>1 0 0</fdir1>
-        </gazebo> -->
-        <gazebo reference="${prefix}chassis_link">
-            <mu1>0.0001</mu1>
-            <mu2>0.0001</mu2>
-        </gazebo>
-        <gazebo reference="${prefix}front_right_wheel_link">
-            <mu1>100.0</mu1>
-            <mu2>100.0</mu2>
-        </gazebo>
-        <gazebo reference="${prefix}front_left_wheel_link">
-            <mu1>100.0</mu1>
-            <mu2>100.0</mu2>
-        </gazebo>
-        <gazebo reference="${prefix}rear_right_wheel_link">
-            <mu1>100.0</mu1>
-            <mu2>100.0</mu2>
-        </gazebo>
-        <gazebo reference="${prefix}rear_left_wheel_link">
-            <mu1>100.0</mu1>
-            <mu2>100.0</mu2>
-        </gazebo>
-        <gazebo reference="${prefix}front_left_steering_link">
-            <mu1>1.0</mu1>
-            <mu2>1.0</mu2>
-        </gazebo>
-        <gazebo reference="${prefix}front_right_steering_link">
-            <mu1>1.0</mu1>
-            <mu2>1.0</mu2>
-        </gazebo>
         <gazebo reference="${prefix}chassis_link">
             <material>Gazebo/Red</material>
         </gazebo>
-        <!-- Gazebo Control -->
         <ros2_control name="${name}" type="system">
             <hardware>
                 <plugin>gazebo_ros2_control/GazeboSystem</plugin>
             </hardware>
-        <joint name="front_left_steering_joint">
-            <command_interface name="position">
-                <param name="min">${-max_steering_angle}</param>
-                <param name="max">${max_steering_angle}</param>
-            </command_interface>
-            <state_interface name="position"/>
-            <state_interface name="velocity"/>
-        </joint>
-        <joint name="front_right_steering_joint">
-            <command_interface name="position">
-                <param name="min">${-max_steering_angle}</param>
-                <param name="max">${max_steering_angle}</param>
-            </command_interface>
-            <state_interface name="position"/>
-            <state_interface name="velocity"/>
-        </joint>
-        <joint name="rear_left_wheel_joint">
-            <command_interface name="velocity">
-                <param name="min">${-max_velocity}</param>
-                <param name="max">${max_velocity}</param>
-            </command_interface>
-            <state_interface name="velocity" />
-            <state_interface name="position" />
-        </joint>
-        <joint name="rear_right_wheel_joint">
-            <command_interface name="velocity">
-                <param name="min">${-max_velocity}</param>
-                <param name="max">${max_velocity}</param>
-            </command_interface>
-            <state_interface name="velocity" />
-            <state_interface name="position" />
-        </joint>
+            <joint name="rear_left_wheel_joint">
+                <command_interface name="velocity" />
+                <state_interface name="velocity" />
+                <state_interface name="position" />
+            </joint>
+            <joint name="rear_right_wheel_joint">
+                <command_interface name="velocity" />
+                <state_interface name="velocity" />
+                <state_interface name="position" />
+            </joint>
+            <joint name="left_wheel_steering_joint">
+                <command_interface name="position" />
+                <state_interface name="position" />
+            </joint>
+            <joint name="right_wheel_steering_joint">
+                <command_interface name="position" />
+                <state_interface name="position" />
+            </joint>
         </ros2_control>
-        <!-- Gazebo Plugin -->
         <gazebo>
             <plugin filename="libgazebo_ros2_control.so" name="gazebo_ros2_control">
-            <robot_param>robot_description</robot_param>
-            <robot_param_node>robot_state_publisher</robot_param_node>
             <parameters>$(find delicar_bringup)/config/gazebo_controllers.yaml</parameters>
-            <!-- <remapping>bicycle_steering_controller/tf_odometry:=odom</remapping> -->
             </plugin>
         </gazebo>

File: delicar_bringup/description/urdf/delicar_description.urdf.xacro (robot description, xacro)
@@ -4,23 +4,23 @@
     <!-- Constants for robot dimensions -->
     <xacro:property name="PI" value="3.1415926535897931"/>
-    <xacro:property name="base_mass" value="4.0" />
-    <xacro:property name="base_width" value="0.3" />
-    <xacro:property name="base_length" value="0.525" />
-    <xacro:property name="base_height" value="0.1" />
-    <xacro:property name="wheelbase" value="0.5" />
-    <xacro:property name="wheeltrack" value="0.3" />
-    <xacro:property name="wheel_mass" value="0.5" />
-    <xacro:property name="wheel_len" value="0.05" />
-    <xacro:property name="wheel_radius" value="0.1" />
+    <xacro:property name="base_mass" value="100.0" />
+    <xacro:property name="base_width" value="1" />
+    <xacro:property name="base_length" value="2" />
+    <xacro:property name="base_height" value="0.5" />
+    <xacro:property name="wheelbase" value="1.6" />
+    <xacro:property name="wheeltrack" value="1.0" />
+    <xacro:property name="wheel_mass" value="11.3" />
+    <xacro:property name="wheel_len" value="0.08" />
+    <xacro:property name="wheel_radius" value="0.3" />
     <!-- Base Link -->
     <link name="${prefix}base_link" />
     <!-- Chassis -->
     <link name="${prefix}chassis_link">
-      <collision>
+      <!-- <collision>
         <origin xyz="0 0 0" rpy="0 0 0"/>
         <geometry>
           <box size="${base_length} ${base_width} ${base_height}"/>
         </geometry>
-      </collision>
+      </collision> -->
       <visual>
         <origin xyz="0 0 0" rpy="0 0 0"/>
@@ -45,44 +45,9 @@
       <parent link="${prefix}base_link"/>
       <child link="${prefix}chassis_link"/>
-      <origin xyz="0 0 ${base_height/2 + wheel_radius}" rpy="0 0 0"/>
+      <origin xyz="0.8 0 0.5" rpy="0 0 0"/>
       <axis xyz="0 0 1"/>
       <dynamics damping="0.2"/>
     </joint>
     <!-- rear wheels -->
-    <!-- rear right wheel -->
-    <link name="${prefix}rear_right_wheel">
-      <collision>
-        <origin xyz="0 0 0" rpy="0 0 0"/>
-        <geometry>
-          <cylinder length="${wheel_len}" radius="${wheel_radius}"/>
-        </geometry>
-      </collision>
-      <visual>
-        <origin xyz="0 0 0" rpy="0 0 0"/>
-        <geometry>
-          <cylinder length="${wheel_len}" radius="${wheel_radius}"/>
-        </geometry>
-        <material name="black"/>
-      </visual>
-      <inertial>
-        <origin xyz="0 0 0" rpy="0 0 0"/>
-        <mass value="${wheel_mass}"/>
-        <inertia
-          ixx="${wheel_mass / 12.0 * (3 * wheel_radius*wheel_radius + wheel_len*wheel_len)}"
-          ixy="0.0"
-          ixz="0.0"
-          iyy="${wheel_mass / 12.0 * (3 * wheel_radius*wheel_radius + wheel_len*wheel_len)}"
-          iyz="0.0"
-          izz="${wheel_mass / 2.0 * wheel_radius*wheel_radius}"/>
-      </inertial>
-    </link>
-    <joint name="${prefix}rear_right_wheel_joint" type="continuous">
-      <parent link="${prefix}chassis_link"/>
-      <child link="${prefix}rear_right_wheel"/>
-      <origin xyz="-${wheelbase/2} ${base_width/2} -${base_height/2}" rpy="-${PI/2} 0 0"/>
-      <axis xyz="0 0 1"/>
-      <limit effort="10.0" velocity="50.0"/>
-      <dynamics damping="0.2"/>
-    </joint>
     <!-- rear left wheel -->
     <link name="${prefix}rear_left_wheel">
@@ -115,16 +80,14 @@
       <parent link="${prefix}chassis_link" />
       <child link="${prefix}rear_left_wheel" />
-      <origin xyz="-${wheelbase/2} -${base_width/2} -${base_height/2}" rpy="-${PI/2} 0 0"/>
-      <axis xyz="0 0 1"/>
-      <limit effort="10.0" velocity="50.0"/>
-      <dynamics damping="0.2"/>
-    </joint>
-    <!-- front steering links-->
-    <!-- front right sterring link-->
-    <link name="${prefix}front_right_steering_link">
+      <origin xyz="-${wheelbase/2} ${wheeltrack/2} -${base_height/2}" rpy="-1.57 0 0"/>
+      <axis xyz="0 0 1"/>
+      <dynamics damping="0.2"/>
+    </joint>
+    <!-- rear right wheel -->
+    <link name="${prefix}rear_right_wheel">
       <collision>
         <origin xyz="0 0 0" rpy="0 0 0"/>
         <geometry>
-          <box size="0.001 0.001 0.001"/>
+          <cylinder length="${wheel_len}" radius="${wheel_radius}"/>
         </geometry>
       </collision>
@@ -132,35 +95,67 @@
         <origin xyz="0 0 0" rpy="0 0 0"/>
         <geometry>
-          <box size="0.001 0.001 0.001"/>
-        </geometry>
-        <material name="invisible"/>
-      </visual>
-      <inertial>
-        <origin xyz="0 0 0" rpy="0 0 0"/>
-        <mass value="0.1"/>
-        <inertia
-          ixx="0.001"
-          ixy="0.0"
-          ixz="0.0"
-          iyy="0.001"
-          iyz="0.0"
-          izz="0.001"/>
-      </inertial>
-    </link>
-    <!-- front right sterring joint-->
-    <joint name="${prefix}front_right_steering_joint" type="revolute">
+          <cylinder length="${wheel_len}" radius="${wheel_radius}"/>
+        </geometry>
+        <material name="black"/>
+      </visual>
+      <inertial>
+        <origin xyz="0 0 0" rpy="0 0 0"/>
+        <mass value="${wheel_mass}"/>
+        <inertia
+          ixx="${wheel_mass / 12.0 * (3 * wheel_radius*wheel_radius + wheel_len*wheel_len)}"
+          ixy="0.0"
+          ixz="0.0"
+          iyy="${wheel_mass / 12.0 * (3 * wheel_radius*wheel_radius + wheel_len*wheel_len)}"
+          iyz="0.0"
+          izz="${wheel_mass / 2.0 * wheel_radius*wheel_radius}"/>
+      </inertial>
+    </link>
+    <joint name="${prefix}rear_right_wheel_joint" type="continuous">
       <parent link="${prefix}chassis_link"/>
-      <child link="${prefix}front_right_steering_link"/>
-      <origin xyz="${wheelbase/2} ${base_width/2} -${base_height/2}" rpy="${PI/2} 0 0"/>
+      <child link="${prefix}rear_right_wheel"/>
+      <origin xyz="-${wheelbase/2} -${wheeltrack/2} -${base_height/2}" rpy="-1.57 0 0"/>
+      <axis xyz="0 0 1"/>
+      <dynamics damping="0.2"/>
+    </joint>
+    <!-- steering links-->
+    <!-- left sterring link-->
+    <link name="${prefix}left_wheel_steering">
+      <inertial>
+      <mass value="0.1"/>
+      <inertia ixx="0.0" ixy="0.0" ixz="0.0" iyy="0.0" iyz="0.0" izz="0.0" />
+      </inertial>
+    </link>
+    <!-- left sterring joint-->
+    <joint name="${prefix}left_wheel_steering_joint" type="revolute">
+      <parent link="${prefix}chassis_link"/>
+      <child link="${prefix}left_wheel_steering"/>
+      <origin xyz="${wheelbase/2} -${wheeltrack/2} -${base_height/2}" rpy="${PI/2} 0 0"/>
       <axis xyz="0 1 0"/>
-      <limit lower="-${PI/4}" upper="${PI/4}" effort="50.0" velocity="1.0"/>
-      <dynamics damping="0.1"/>
-    </joint>
-    <!-- front left sterring link-->
-    <link name="${prefix}front_left_steering_link">
+      <dynamics damping="0.2"/>
+      <limit effort="1000.0" lower="-1.0471975512" upper="1.0471975512" velocity="30"/>
+    </joint>
+    <!-- right sterring link-->
+    <link name="${prefix}right_wheel_steering">
+      <inertial>
+      <mass value="0.1"/>
+      <inertia ixx="0.0" ixy="0.0" ixz="0.0" iyy="0.0" iyz="0.0" izz="0.0" />
+      </inertial>
+    </link>
+    <!-- right sterring joint-->
+    <joint name="${prefix}right_wheel_steering_joint" type="revolute">
+      <parent link="${prefix}chassis_link"/>
+      <child link="${prefix}right_wheel_steering"/>
+      <origin xyz="${wheelbase/2} ${wheeltrack/2} -${base_height/2}" rpy="${PI/2} 0 0"/>
+      <axis xyz="0 1 0"/>
+      <dynamics damping="0.2"/>
+      <limit effort="1000.0" lower="-1.0471975512" upper="1.0471975512" velocity="30"/>
+    </joint>
+    <!-- front wheels -->
+    <!-- front left steering -->
+    <link name="${prefix}front_left_wheel">
       <collision>
         <origin xyz="0 0 0" rpy="0 0 0"/>
         <geometry>
-          <box size="0.001 0.001 0.001"/>
+          <cylinder length="${wheel_len}" radius="${wheel_radius}"/>
         </geometry>
       </collision>
@@ -168,30 +163,27 @@
         <origin xyz="0 0 0" rpy="0 0 0"/>
         <geometry>
-          <box size="0.001 0.001 0.001"/>
-        </geometry>
-        <material name="invisible"/>
-      </visual>
-      <inertial>
-        <origin xyz="0 0 0" rpy="0 0 0"/>
-        <mass value="0.1"/>
-        <inertia
-          ixx="0.001"
-          ixy="0.0"
-          ixz="0.0"
-          iyy="0.001"
-          iyz="0.0"
-          izz="0.001"/>
-      </inertial>
-    </link>
-    <!-- front left sterring joint-->
-    <joint name="${prefix}front_left_steering_joint" type="revolute">
-      <parent link="${prefix}chassis_link"/>
-      <child link="${prefix}front_left_steering_link"/>
-      <origin xyz="${wheelbase/2} -${base_width/2} -${base_height/2}" rpy="${PI/2} 0 0"/>
-      <axis xyz="0 1 0"/>
-      <limit lower="-${PI/4}" upper="${PI/4}" effort="50.0" velocity="1.0"/>
-      <dynamics damping="0.1"/>
-    </joint>
-    <!-- front wheels -->
+          <cylinder length="${wheel_len}" radius="${wheel_radius}"/>
+        </geometry>
+        <material name="black"/>
+      </visual>
+      <inertial>
+        <origin xyz="0 0 0" rpy="0 0 0"/>
+        <mass value="${wheel_mass}"/>
+        <inertia
+          ixx="${wheel_mass / 12.0 * (3 * wheel_radius*wheel_radius + wheel_len*wheel_len)}"
+          ixy="0.0"
+          ixz="0.0"
+          iyy="${wheel_mass / 12.0 * (3 * wheel_radius*wheel_radius + wheel_len*wheel_len)}"
+          iyz="0.0"
+          izz="${wheel_mass / 2.0 * wheel_radius*wheel_radius}"/>
+      </inertial>
+    </link>
+    <joint name="${prefix}front_left_wheel_joint" type="continuous">
+      <parent link="${prefix}left_wheel_steering" />
+      <child link="${prefix}front_left_wheel" />
+      <origin xyz="0 0 0" rpy="0 0 0"/>
+      <axis xyz="0 0 1"/>
+      <dynamics damping="0.2"/>
+    </joint>
     <!-- front right wheel -->
     <link name="${prefix}front_right_wheel">
@@ -222,44 +214,8 @@
     </link>
     <joint name="${prefix}front_right_wheel_joint" type="continuous">
-      <parent link="${prefix}front_right_steering_link" />
+      <parent link="${prefix}right_wheel_steering" />
       <child link="${prefix}front_right_wheel" />
       <origin xyz="0 0 0" rpy="0 0 0"/>
       <axis xyz="0 0 1"/>
-      <limit effort="10.0" velocity="50.0"/>
-      <dynamics damping="0.2"/>
-    </joint>
-    <!-- front left steering -->
-    <link name="${prefix}front_left_wheel">
-      <collision>
-        <origin xyz="0 0 0" rpy="0 0 0"/>
-        <geometry>
-          <cylinder length="${wheel_len}" radius="${wheel_radius}"/>
-        </geometry>
-      </collision>
-      <visual>
-        <origin xyz="0 0 0" rpy="0 0 0"/>
-        <geometry>
-          <cylinder length="${wheel_len}" radius="${wheel_radius}"/>
-        </geometry>
-        <material name="black"/>
-      </visual>
-      <inertial>
-        <origin xyz="0 0 0" rpy="0 0 0"/>
-        <mass value="${wheel_mass}"/>
-        <inertia
-          ixx="${wheel_mass / 12.0 * (3 * wheel_radius*wheel_radius + wheel_len*wheel_len)}"
-          ixy="0.0"
-          ixz="0.0"
-          iyy="${wheel_mass / 12.0 * (3 * wheel_radius*wheel_radius + wheel_len*wheel_len)}"
-          iyz="0.0"
-          izz="${wheel_mass / 2.0 * wheel_radius*wheel_radius}"/>
-      </inertial>
-    </link>
-    <joint name="${prefix}front_left_wheel_joint" type="continuous">
-      <parent link="${prefix}front_left_steering_link" />
-      <child link="${prefix}front_left_wheel" />
-      <origin xyz="0 0 0" rpy="0 0 0"/>
-      <axis xyz="0 0 1"/>
-      <limit effort="10.0" velocity="50.0"/>
       <dynamics damping="0.2"/>
     </joint>
