Commit message: Create gazebo simulation

File: delicar_bringup/description/urdf/delicar.urdf.xacro (robot description, xacro)
@@ -3,11 +3,18 @@
 <robot xmlns:xacro="http://www.ros.org/wiki/xacro" name="delicar_robot">
   <xacro:arg name="prefix" default="" />
+  <xacro:arg name="use_sim" default="true"/>
   <xacro:include filename="$(find delicar_bringup)/urdf/delicar_description.urdf.xacro" />
-  <!-- Import Rviz colors -->
+  <!-- Import colors -->
   <xacro:include filename="$(find delicar_bringup)/urdf/color.materials.xacro" />
-  <!-- Import delicar ros2_control description -->
-  <xacro:include filename="$(find delicar_bringup)/ros2_control/delicar.ros2_control.xacro" />
-  <xacro:delicar prefix="$(arg prefix)" />
-  <xacro:delicar_ros2_control
-    name="DeliCar" prefix="$(arg prefix)" />
+  <!-- Import delicar description -->
+  <xacro:delicar prefix="" />
+  <!-- Import delicar ros2_control -->
+  <xacro:unless value="$(arg use_sim)">
+    <xacro:include filename="$(find delicar_bringup)/ros2_control/delicar_controllers.xacro" />
+    <xacro:delicar_ros2_control name="DeliCar" prefix="$(arg prefix)" />
+  </xacro:unless>
+  <xacro:if value="$(arg use_sim)">
+    <xacro:include filename="$(find delicar_bringup)/ros2_control/gazebo_controllers.xacro" />
+    <xacro:gazebo_ros2_control name="GazeboSystem" prefix="$(arg prefix)" />
+  </xacro:if>
 </robot>

File: delicar_bringup/description/urdf/delicar_description.urdf.xacro (robot description, xacro)
@@ -2,39 +2,42 @@
 <robot xmlns:xacro="http://www.ros.org/wiki/xacro">
   <xacro:macro name="delicar" params="prefix">
-  <!-- Constants for robot dimensions -->
-  <xacro:property name="PI" value="3.1415926535897931"/>
-  <xacro:property name="base_mass" value="4.0" />
-  <xacro:property name="base_width" value="0.260" />
-  <xacro:property name="base_length" value="0.525" />
-  <xacro:property name="base_height" value="0.060" />
-  <xacro:property name="wheelbase" value="0.325" />
-  <xacro:property name="wheel_mass" value="0.34055" />
-  <xacro:property name="wheel_len" value="0.045" />
-  <xacro:property name="wheel_radius" value="0.05" />
-  <!-- <xacro:property name="wheeltrack" value="" -->
-  <!-- Base Link -->
-  <link name="${prefix}base_link" />
-  <!-- Chassis -->
-  <link name="${prefix}chassis_link">
-    <collision>
-      <origin xyz="0 0 0" rpy="0 0 0"/>
-      <geometry>
-        <box size="${base_length} ${base_width} ${base_height}"/>
-      </geometry>
-    </collision>
-    <visual>
-      <origin xyz="0 0 0" rpy="0 0 0"/>
-      <geometry>
-        <box size="${base_length} ${base_width} ${base_height}"/>
-      </geometry>
-      <material name="orange"/>
-    </visual>
-    <inertial>
-      <origin xyz="0 0 0" rpy="0 0 0"/>
-      <mass value="${base_mass}"/>
-        <inertia
-          ixx="0.000270" ixy="0.0" ixz="0.0"
-          iyy="0.000270" iyz="0.0"
-          izz="0.000426"/>
+    <!-- Constants for robot dimensions -->
+    <xacro:property name="PI" value="3.1415926535897931"/>
+    <xacro:property name="base_mass" value="4.0" />
+    <xacro:property name="base_width" value="0.3" />
+    <xacro:property name="base_length" value="0.525" />
+    <xacro:property name="base_height" value="0.1" />
+    <xacro:property name="wheelbase" value="0.5" />
+    <xacro:property name="wheeltrack" value="0.3" />
+    <xacro:property name="wheel_mass" value="0.5" />
+    <xacro:property name="wheel_len" value="0.05" />
+    <xacro:property name="wheel_radius" value="0.1" />
+    <!-- Base Link -->
+    <link name="${prefix}base_link" />
+    <!-- Chassis -->
+    <link name="${prefix}chassis_link">
+      <collision>
+        <origin xyz="0 0 0" rpy="0 0 0"/>
+        <geometry>
+          <box size="${base_length} ${base_width} ${base_height}"/>
+        </geometry>
+      </collision>
+      <visual>
+        <origin xyz="0 0 0" rpy="0 0 0"/>
+        <geometry>
+          <box size="${base_length} ${base_width} ${base_height}"/>
+        </geometry>
+        <material name="orange"/>
+      </visual>
+      <inertial>
+        <origin xyz="0 0 0" rpy="0 0 0"/>
+        <mass value="${base_mass}"/>
+        <inertia
+          ixx="${base_mass / 12.0 * (base_width*base_width + base_height*base_height)}"
+          ixy="0.0"
+          ixz="0.0"
+          iyy="${base_mass / 12.0 * (base_width*base_width + base_height*base_height)}"
+          iyz="0.0"
+          izz="${base_mass / 12.0 * (base_width*base_width + base_height*base_height)}"/>
       </inertial>
     </link>
@@ -47,22 +50,4 @@
     </joint>
     <!-- rear wheels -->
-    <!-- virtual rear wheel -->
-    <link name="${prefix}virtual_rear_wheel">
-      <visual>
-        <origin xyz="0 0 0" rpy="${PI/2} 0 ${PI/2}"/>
-        <geometry>
-          <cylinder length="0.01" radius="${wheel_radius}"/>
-        </geometry>
-        <material name="invisible"/>
-      </visual>
-    </link>
-    <joint name="${prefix}virtual_rear_wheel_joint" type="continuous">
-      <parent link="${prefix}chassis_link"/>
-      <child link="${prefix}virtual_rear_wheel"/>
-      <origin xyz="-${wheelbase/2} 0 -${base_height/2}" rpy="0 0 ${PI/2}"/>
-      <axis xyz="1 0 0"/>
-      <limit effort="100.0" velocity="100.0"/>
-      <dynamics damping="0.2"/>
-    </joint>
     <!-- rear right wheel -->
     <link name="${prefix}rear_right_wheel">
@@ -84,7 +69,10 @@
         <mass value="${wheel_mass}"/>
         <inertia
-          ixx="0.000270" ixy="0.0" ixz="0.0"
-          iyy="0.000270" iyz="0.0"
-          izz="0.000426"/>
+          ixx="${wheel_mass / 12.0 * (3 * wheel_radius*wheel_radius + wheel_len*wheel_len)}"
+          ixy="0.0"
+          ixz="0.0"
+          iyy="${wheel_mass / 12.0 * (3 * wheel_radius*wheel_radius + wheel_len*wheel_len)}"
+          iyz="0.0"
+          izz="${wheel_mass / 2.0 * wheel_radius*wheel_radius}"/>
       </inertial>
     </link>
@@ -94,7 +82,6 @@
       <origin xyz="-${wheelbase/2} ${base_width/2} -${base_height/2}" rpy="0 0 ${PI/2}"/>
       <axis xyz="1 0 0"/>
-      <limit effort="100.0" velocity="100.0"/>
-      <dynamics damping="0.2"/>
-      <mimic joint="${prefix}virtual_rear_wheel_joint" multiplier="1.0" offset="0.0"/>
+      <limit effort="10.0" velocity="50.0"/>
+      <dynamics damping="0.2"/>
     </joint>
     <!-- rear left wheel -->
@@ -117,7 +104,10 @@
           <mass value="${wheel_mass}"/>
           <inertia
-            ixx="0.000270" ixy="0.0" ixz="0.0"
-            iyy="0.000270" iyz="0.0"
-            izz="0.000426"/>
+            ixx="${wheel_mass / 12.0 * (3 * wheel_radius*wheel_radius + wheel_len*wheel_len)}"
+            ixy="0.0"
+            ixz="0.0"
+            iyy="${wheel_mass / 12.0 * (3 * wheel_radius*wheel_radius + wheel_len*wheel_len)}"
+            iyz="0.0"
+            izz="${wheel_mass / 2.0 * wheel_radius*wheel_radius}"/>
         </inertial>
     </link>
@@ -127,27 +117,81 @@
       <origin xyz="-${wheelbase/2} -${base_width/2} -${base_height/2}" rpy="0 0 ${PI/2}"/>
       <axis xyz="1 0 0"/>
-      <limit effort="100.0" velocity="100.0"/>
-      <dynamics damping="0.2"/>
-      <mimic joint="${prefix}virtual_rear_wheel_joint" multiplier="1.0" offset="0.0"/>
+      <limit effort="10.0" velocity="50.0"/>
+      <dynamics damping="0.2"/>
+    </joint>
+    <!-- front steering links-->
+    <!-- front right sterring link-->
+    <link name="${prefix}front_right_steering_link">
+      <collision>
+        <origin xyz="0 0 0" rpy="0 0 0"/>
+        <geometry>
+          <box size="0.001 0.001 0.001"/>
+        </geometry>
+      </collision>
+      <visual>
+        <origin xyz="0 0 0" rpy="0 0 0"/>
+        <geometry>
+          <box size="0.001 0.001 0.001"/>
+        </geometry>
+        <material name="invisible"/>
+      </visual>
+      <inertial>
+        <origin xyz="0 0 0" rpy="0 0 0"/>
+        <mass value="0.1"/>
+        <inertia
+          ixx="0.001"
+          ixy="0.0"
+          ixz="0.0"
+          iyy="0.001"
+          iyz="0.0"
+          izz="0.001"/>
+      </inertial>
+    </link>
+    <!-- front right sterring joint-->
+    <joint name="${prefix}front_right_steering_joint" type="revolute">
+      <parent link="${prefix}chassis_link"/>
+      <child link="${prefix}front_right_steering_link"/>
+      <origin xyz="${wheelbase/2} ${base_width/2} -${base_height/2}" rpy="0 0 0"/>
+      <axis xyz="0 0 1"/>
+      <limit lower="-${PI/4}" upper="${PI/4}" effort="50.0" velocity="1.0"/>
+      <dynamics damping="0.1"/>
+    </joint>
+    <!-- front left sterring link-->
+    <link name="${prefix}front_left_steering_link">
+      <collision>
+        <origin xyz="0 0 0" rpy="0 0 0"/>
+        <geometry>
+          <box size="0.001 0.001 0.001"/>
+        </geometry>
+      </collision>
+      <visual>
+        <origin xyz="0 0 0" rpy="0 0 0"/>
+        <geometry>
+          <box size="0.001 0.001 0.001"/>
+        </geometry>
+        <material name="invisible"/>
+      </visual>
+      <inertial>
+        <origin xyz="0 0 0" rpy="0 0 0"/>
+        <mass value="0.1"/>
+        <inertia
+          ixx="0.001"
+          ixy="0.0"
+          ixz="0.0"
+          iyy="0.001"
+          iyz="0.0"
+          izz="0.001"/>
+      </inertial>
+    </link>
+    <!-- front left sterring joint-->
+    <joint name="${prefix}front_left_steering_joint" type="revolute">
+      <parent link="${prefix}chassis_link"/>
+      <child link="${prefix}front_left_steering_link"/>
+      <origin xyz="${wheelbase/2} -${base_width/2} -${base_height/2}" rpy="0 0 0"/>
+      <axis xyz="0 0 1"/>
+      <limit lower="-${PI/4}" upper="${PI/4}" effort="50.0" velocity="1.0"/>
+      <dynamics damping="0.1"/>
     </joint>
     <!-- front wheels -->
-    <!-- virtual front wheel -->
-    <link name="${prefix}virtual_front_wheel">
-      <visual>
-        <origin xyz="0 0 0" rpy="${PI/2} 0 ${PI/2}"/>
-        <geometry>
-          <cylinder length="0.01" radius="${wheel_radius}"/>
-        </geometry>
-        <material name="invisible"/>
-      </visual>
-    </link>
-    <joint name="${prefix}virtual_front_wheel_joint" type="revolute">
-      <parent link="${prefix}chassis_link"/>
-      <child link="${prefix}virtual_front_wheel"/>
-      <origin xyz="${wheelbase/2} 0 -${base_height/2}" rpy="0 0 ${PI/2}"/>
-      <axis xyz="0 0 1"/>
-      <limit lower="-0.4" upper="0.4" effort="100.0" velocity="0.0"/>
-      <dynamics damping="0.2"/>
-    </joint>
     <!-- front right wheel -->
     <link name="${prefix}front_right_wheel">
@@ -169,17 +213,19 @@
         <mass value="${wheel_mass}"/>
         <inertia
-          ixx="0.000270" ixy="0.0" ixz="0.0"
-          iyy="0.000270" iyz="0.0"
-          izz="0.000426"/>
-      </inertial>
-    </link>
-    <joint name="${prefix}front_right_wheel_joint" type="revolute">
-      <parent link="${prefix}chassis_link" />
+          ixx="${wheel_mass / 12.0 * (3 * wheel_radius*wheel_radius + wheel_len*wheel_len)}"
+          ixy="0.0"
+          ixz="0.0"
+          iyy="${wheel_mass / 12.0 * (3 * wheel_radius*wheel_radius + wheel_len*wheel_len)}"
+          iyz="0.0"
+          izz="${wheel_mass / 2.0 * wheel_radius*wheel_radius}"/>
+      </inertial>
+    </link>
+    <joint name="${prefix}front_right_wheel_joint" type="continuous">
+      <parent link="${prefix}front_right_steering_link" />
       <child link="${prefix}front_right_wheel" />
-      <origin xyz="${wheelbase/2} ${base_width/2} -${base_height/2}" rpy="0 0 ${PI/2}"/>
-      <axis xyz="0 0 1"/>
-      <limit lower="-0.4" upper="0.4" effort="100.0" velocity="0.0"/>
-      <dynamics damping="0.2"/>
-      <mimic joint="${prefix}virtual_front_wheel_joint" multiplier="1.0" offset="0.0"/>
+      <origin xyz="0 0 0" rpy="0 0 ${PI/2}"/>
+      <axis xyz="1 0 0"/>
+      <limit effort="10.0" velocity="50.0"/>
+      <dynamics damping="0.2"/>
     </joint>
     <!-- front left steering -->
@@ -202,17 +248,19 @@
         <mass value="${wheel_mass}"/>
         <inertia
-          ixx="0.000270" ixy="0.0" ixz="0.0"
-          iyy="0.000270" iyz="0.0"
-          izz="0.000426"/>
-      </inertial>
-    </link>
-    <joint name="${prefix}front_left_wheel_joint" type="revolute">
-      <parent link="${prefix}chassis_link" />
+          ixx="${wheel_mass / 12.0 * (3 * wheel_radius*wheel_radius + wheel_len*wheel_len)}"
+          ixy="0.0"
+          ixz="0.0"
+          iyy="${wheel_mass / 12.0 * (3 * wheel_radius*wheel_radius + wheel_len*wheel_len)}"
+          iyz="0.0"
+          izz="${wheel_mass / 2.0 * wheel_radius*wheel_radius}"/>
+      </inertial>
+    </link>
+    <joint name="${prefix}front_left_wheel_joint" type="continuous">
+      <parent link="${prefix}front_left_steering_link" />
       <child link="${prefix}front_left_wheel" />
-      <origin xyz="${wheelbase/2} -${base_width/2} -${base_height/2}" rpy="0 0 ${PI/2}"/>
-      <axis xyz="0 0 1"/>
-      <limit lower="-0.4" upper="0.4" effort="100.0" velocity="0.0"/>
-      <dynamics damping="0.2"/>
-      <mimic joint="${prefix}virtual_front_wheel_joint" multiplier="1.0" offset="0.0"/>
+      <origin xyz="0 0 0" rpy="0 0 ${PI/2}"/>
+      <axis xyz="1 0 0"/>
+      <limit effort="10.0" velocity="50.0"/>
+      <dynamics damping="0.2"/>
     </joint>
   </xacro:macro>

Commit message: Add IMU

File: delicar_bringup/description/urdf/delicar.urdf.xacro (robot description, xacro)
@@ -10,4 +10,7 @@
   <xacro:include filename="$(find delicar_bringup)/urdf/camera.urdf.xacro" />
   <xacro:camera prefix="$(arg prefix)" />
+  <!-- Import imu -->
+  <xacro:include filename="$(find delicar_bringup)/urdf/imu.urdf.xacro" />
+  <xacro:imu prefix="$(arg prefix)" />
   <!-- Import delicar description -->
   <xacro:delicar prefix="" />

File: delicar_bringup/description/urdf/imu.urdf.xacro (robot description, xacro)
@@ -1,5 +1,103 @@
 <?xml version="1.0"?>
 <robot xmlns:xacro="http://www.ros.org/wiki/xacro">
-  <xacro:macro name="imu" params="prefix">
-  </xacro:macro>
+    <xacro:macro name="imu" params="prefix">
+        <xacro:macro name="box_inertia" params="m w h d">
+            <inertial>
+                <origin xyz="0 0 0" rpy="${pi/2} 0 ${pi/2}" />
+                <mass value="${m}" />
+                <inertia ixx="${(m/12) * (h*h + d*d)}" ixy="0.0" ixz="0.0"
+                    iyy="${(m/12) * (w*w + d*d)}" iyz="0.0" izz="${(m/12) * (w*w + h*h)}" />
+            </inertial>
+        </xacro:macro>
+        <xacro:macro name="cylinder_inertia" params="m r h">
+            <inertial>
+                <origin xyz="0 0 0" rpy="${pi/2} 0 0" />
+                <mass value="${m}" />
+                <inertia ixx="${(m/12) * (3*r*r + h*h)}" ixy="0" ixz="0"
+                    iyy="${(m/12) * (3*r*r + h*h)}" iyz="0" izz="${(m/2) * (r*r)}" />
+            </inertial>
+        </xacro:macro>
+        <xacro:macro name="sphere_inertia" params="m r">
+            <inertial>
+                <mass value="${m}" />
+                <inertia ixx="${(2/5) * m * (r*r)}" ixy="0.0" ixz="0.0" iyy="${(2/5) * m * (r*r)}"
+                    iyz="0.0" izz="${(2/5) * m * (r*r)}" />
+            </inertial>
+        </xacro:macro>
+        <link name="imu_link">
+            <xacro:box_inertia m="0.1" w="0.1" d="0.1" h="0.1" />
+        </link>
+        <joint name="${prefix}imu_joint" type="fixed">
+            <parent link="${prefix}base_link" />
+            <child link="${prefix}imu_link" />
+            <origin xyz="0 0 0.01" />
+        </joint>
+        <gazebo reference="${prefix}imu_link">
+            <sensor name="imu_sensor" type="imu">
+                <plugin filename="libgazebo_ros_imu_sensor.so" name="imu_plugin">
+                    <ros>
+                        <remapping>~/out:=imu_raw</remapping>
+                    </ros>
+                    <initial_orientation_as_reference>false</initial_orientation_as_reference>
+                </plugin>
+                <always_on>true</always_on>
+                <update_rate>100</update_rate>
+                <visualize>true</visualize>
+                <imu>
+                    <angular_velocity>
+                        <x>
+                            <noise type="gaussian">
+                                <mean>0.0</mean>
+                                <stddev>2e-4</stddev>
+                                <bias_mean>0.0000075</bias_mean>
+                                <bias_stddev>0.0000008</bias_stddev>
+                            </noise>
+                        </x>
+                        <y>
+                            <noise type="gaussian">
+                                <mean>0.0</mean>
+                                <stddev>2e-4</stddev>
+                                <bias_mean>0.0000075</bias_mean>
+                                <bias_stddev>0.0000008</bias_stddev>
+                            </noise>
+                        </y>
+                        <z>
+                            <noise type="gaussian">
+                                <mean>0.0</mean>
+                                <stddev>2e-4</stddev>
+                                <bias_mean>0.0000075</bias_mean>
+                                <bias_stddev>0.0000008</bias_stddev>
+                            </noise>
+                        </z>
+                    </angular_velocity>
+                    <linear_acceleration>
+                        <x>
+                            <noise type="gaussian">
+                                <mean>0.0</mean>
+                                <stddev>1.7e-2</stddev>
+                                <bias_mean>0.1</bias_mean>
+                                <bias_stddev>0.001</bias_stddev>
+                            </noise>
+                        </x>
+                        <y>
+                            <noise type="gaussian">
+                                <mean>0.0</mean>
+                                <stddev>1.7e-2</stddev>
+                                <bias_mean>0.1</bias_mean>
+                                <bias_stddev>0.001</bias_stddev>
+                            </noise>
+                        </y>
+                        <z>
+                            <noise type="gaussian">
+                                <mean>0.0</mean>
+                                <stddev>1.7e-2</stddev>
+                                <bias_mean>0.1</bias_mean>
+                                <bias_stddev>0.001</bias_stddev>
+                            </noise>
+                        </z>
+                    </linear_acceleration>
+                </imu>
+            </sensor>
+        </gazebo>
+    </xacro:macro>
 </robot>
