Commit message: Add velodyne 3D lidar

File: delicar_bringup/description/urdf/color.materials.xacro (robot description, xacro)
@@ -1,34 +1,35 @@
 <?xml version="1.0"?>
-<!--
-Copied from ROS1 example:
-https://github.com/ros-simulation/gazebo_ros_demos/blob/kinetic-devel/rrbot_description/urdf/materials.xacro
--->
-<robot>
+<robot name="xacro_properties"
+  xmlns:xacro="http://ros.org/wiki/xacro">
+  <!-- Init colour -->
   <material name="black">
-    <color rgba="0.0 0.0 0.0 1.0"/>
+    <color rgba="0.0 0.0 0.0 1.0" />
+  </material>
+  <material name="dark">
+    <color rgba="0.3 0.3 0.3 1.0" />
+  </material>
+  <material name="light_black">
+    <color rgba="0.4 0.4 0.4 1.0" />
   </material>
   <material name="blue">
-    <color rgba="0.0 0.0 0.8 1.0"/>
+    <color rgba="0.0 0.0 0.8 1.0" />
   </material>
   <material name="green">
-    <color rgba="0.0 0.8 0.0 1.0"/>
+    <color rgba="0.0 0.8 0.0 1.0" />
   </material>
   <material name="grey">
-    <color rgba="0.2 0.2 0.2 1.0"/>
+    <color rgba="0.5 0.5 0.5 1.0" />
   </material>
   <material name="orange">
-    <color rgba="${255/255} ${108/255} ${10/255} 1.0"/>
+    <color rgba="${255/255} ${108/255} ${10/255} 1.0" />
   </material>
   <material name="brown">
-    <color rgba="${222/255} ${207/255} ${195/255} 1.0"/>
+    <color rgba="${222/255} ${207/255} ${195/255} 1.0" />
   </material>
   <material name="red">
-    <color rgba="0.8 0.0 0.0 1.0"/>
+    <color rgba="0.8 0.0 0.0 1.0" />
   </material>
   <material name="white">
-    <color rgba="1.0 1.0 1.0 1.0"/>
-  </material>
-  <material name="invisible">
-    <color rgba="0.0 0.0 0.0 0.0"/>
+    <color rgba="1.0 1.0 1.0 1.0" />
   </material>
 </robot>

File: delicar_bringup/description/urdf/delicar.urdf.xacro (robot description, xacro)
@@ -4,7 +4,9 @@
   <xacro:arg name="prefix" default="" />
   <xacro:arg name="use_sim" default="true"/>
-  <xacro:include filename="$(find delicar_bringup)/urdf/delicar_description.urdf.xacro" />
   <!-- Import colors -->
   <xacro:include filename="$(find delicar_bringup)/urdf/color.materials.xacro" />
+  <!-- Import delicar description -->
+  <xacro:include filename="$(find delicar_bringup)/urdf/delicar_description.urdf.xacro" />
+  <xacro:delicar prefix="" />
   <!-- Import camera -->
   <xacro:include filename="$(find delicar_bringup)/urdf/camera.urdf.xacro" />
@@ -13,6 +15,7 @@
   <xacro:include filename="$(find delicar_bringup)/urdf/imu.urdf.xacro" />
   <xacro:imu prefix="$(arg prefix)" />
-  <!-- Import delicar description -->
-  <xacro:delicar prefix="" />
+  <!-- Import velodyne lidar -->
+  <xacro:include filename="$(find delicar_bringup)/urdf/velodyne_lidar.urdf.xacro" />
+  <xacro:lidar prefix="$(arg prefix)" />
   <!-- Import delicar ros2_control -->
   <xacro:unless value="$(arg use_sim)">

File: delicar_bringup/description/urdf/imu.urdf.xacro (robot description, xacro)
@@ -26,5 +26,5 @@
         </xacro:macro>
         <link name="imu_link">
-            <xacro:box_inertia m="0.1" w="0.1" d="0.1" h="0.1" />
+            <xacro:box_inertia m="0.01" w="0.01" d="0.01" h="0.01" />
         </link>
         <joint name="${prefix}imu_joint" type="fixed">
