Commit message: Change color of lidar in gazebo

File: delicar_bringup/description/urdf/velodyne_lidar.urdf.xacro (robot description, xacro)
@@ -24,4 +24,5 @@
     </link>
     <gazebo reference="velodyne">
+      <material>Gazebo/Gray</material>
       <sensor name="velodyne-VLP16" type="ray">
         <visualize>false</visualize>
