Commit message: Update navigation package

File: delicar_description/urdf/robot/delicar_description.urdf.xacro (robot description, xacro)
@@ -13,11 +13,4 @@
     <xacro:property name="wheel_len" value="0.1" />
     <xacro:property name="wheel_radius" value="0.225" />
-    <!-- Base footprint -->
-    <link name="${prefix}base_footprint" />
-    <joint name="${prefix}base_to_footprint" type="fixed">
-      <parent link="${prefix}base_footprint" />
-      <child link="${prefix}base_link" />
-      <origin xyz="0 0 ${wheel_radius + base_height/2}" rpy="0 0 0" />
-    </joint>
     <!-- Base Link -->
     <link name="${prefix}base_link" />
@@ -66,5 +59,5 @@
       <parent link="${prefix}base_link" />
       <child link="${prefix}chassis_link" />
-      <origin xyz="0 0 0" rpy="0 0 0" />
+      <origin xyz="0 0 ${wheel_radius + base_height/2}" rpy="0 0 0" />
     </joint>
     <!-- Rear wheels -->

File: delicar_description/urdf/sensors/camera.urdf.xacro (robot description, xacro)
@@ -28,5 +28,5 @@
     <joint name="${prefix}camera_joint" type="fixed">
       <origin
-        xyz="1.8 0 0.7"
+        xyz="1.8 0 1.125"
         rpy="0 0 0" />
       <parent link="${prefix}base_link" />

File: delicar_description/urdf/sensors/depth_camera.urdf.xacro (robot description, xacro)
@@ -28,5 +28,5 @@
     <joint name="${prefix}depth_camera_joint" type="fixed">
         <origin
-        xyz="0.815 0 0.1"
+        xyz="0.815 0 0.525"
         rpy="0 0 0" />
         <parent link="${prefix}base_link" />

File: delicar_description/urdf/sensors/imu.urdf.xacro (robot description, xacro)
@@ -5,5 +5,5 @@
       <parent link="${prefix}base_link" />
       <child link="${prefix}imu_link" />
-      <origin xyz="0 0 0" rpy="0 0 0" />
+      <origin xyz="0 0 0.425" rpy="0 0 0" />
     </joint>
     <gazebo reference="${prefix}imu_link">

File: delicar_description/urdf/sensors/laser_3d.urdf.xacro (robot description, xacro)
@@ -30,5 +30,5 @@
       <parent link="${prefix}base_link" />
       <child link="${frame_id}" />
-      <origin xyz="0.6 0 0.265" rpy="0 0 0" />
+      <origin xyz="0.6 0 0.69" rpy="0 0 0" />
     </joint>
     <gazebo reference="${frame_id}">
