Commit message: Refactoring the code. It happen twice which is strange but it happen

File: delicar_description/urdf/controllers/delicar_controllers.xacro (robot description, xacro)
@@ -4,7 +4,19 @@
     <ros2_control name="${name}" type="system">
       <hardware>
-        <plugin>delicar_bringup/DeliCarSystemHardware</plugin>
-        <param name="hw_start_duration_sec">0</param>
-        <param name="hw_stop_duration_sec">3.0</param>
+        <plugin>delicar_bringup/CarlikeBotSystemHardware</plugin>
+        <param name="drive_wheel_name">virtual_rear_wheel_joint</param>
+        <param name="steer_wheel_name">virtual_front_wheel_joint</param>
+        <param name="serial_port">/dev/ttyUSB0</param>
+        <param name="baud_rate">9600</param>
+        <param name="parity">O</param>
+        <param name="data_bits">8</param>
+        <param name="stop_bits">1</param>
+        <param name="slave_id">1</param>
+        <param name="traction_speed_cmd_register">0</param>
+        <param name="traction_speed_fb_register">2</param>
+        <param name="steering_angle_cmd_register">1</param>
+        <param name="steering_angle_fb_register">6</param>
+        <param name="steering_scale_factor">327.4</param>
+        <param name="traction_scale_factor">1</param>
       </hardware>
       <joint name="${prefix}virtual_front_wheel_joint">

File: delicar_description/urdf/delicar.urdf.xacro (robot description, xacro)
@@ -3,38 +3,23 @@
 <robot xmlns:xacro="http://www.ros.org/wiki/xacro" name="delicar_robot">
   <xacro:arg name="prefix" default="" />
-  <xacro:arg name="use_sim" default="true" />
+  <xacro:arg name="use_sim" default="false" />
+  <xacro:include filename="$(find delicar_description)/urdf/robot/color.materials.xacro" />
   <xacro:include filename="$(find delicar_description)/urdf/robot/delicar_description.urdf.xacro" />
-  <xacro:include filename="$(find delicar_description)/urdf/sensors/depth_camera.urdf.xacro" />
+  <!-- <xacro:include filename="$(find delicar_description)/urdf/sensors/depth_camera.urdf.xacro" /> -->
   <xacro:include filename="$(find delicar_description)/urdf/sensors/imu.urdf.xacro" />
-  <xacro:include filename="$(find delicar_description)/urdf/sensors/laser_3d.urdf.xacro" />
+  <xacro:include filename="$(find delicar_description)/urdf/sensors/lidar_3d.urdf.xacro" />
   <xacro:include filename="$(find delicar_description)/urdf/controllers/delicar_controllers.xacro" />
-  <xacro:include filename="$(find delicar_description)/urdf/controllers/gazebo_controllers.xacro" />
   <!-- Import delicar description -->
   <xacro:delicar prefix="$(arg prefix)" />
   <!-- Import camera -->
-  <xacro:depth_camera prefix="$(arg prefix)" />
+  <!-- <xacro:depth_camera prefix="$(arg prefix)" /> -->
   <!-- Import imu -->
   <xacro:imu prefix="$(arg prefix)"/>
   <!-- Import 3d lidar -->
-  <xacro:laser_3d
+  <xacro:lidar_3d
     prefix="$(arg prefix)"
-    update_rate="10"
-    ray_count="440"
-    line_count="16"
-    hor_min_angle="-3.14159"
-    hor_max_angle="3.14159"
-    ver_min_angle="-0.2617"
-    ver_max_angle="0.2617"
-    min_range="0.3"
-    max_range="130.0"
-    frame_id="laser_3d"
-    topic_name="lidar/points_raw"
+    frame_id="rslidar"
   />
   <!-- Import controllers -->
-  <xacro:unless value="$(arg use_sim)">
-    <xacro:delicar_ros2_control name="DeliCar" prefix="$(arg prefix)" />
-  </xacro:unless>
-  <xacro:if value="$(arg use_sim)">
-    <xacro:gazebo_ros2_control name="GazeboSystem" prefix="$(arg prefix)" />
-  </xacro:if>
+  <xacro:delicar_ros2_control name="Delicar" prefix="$(arg prefix)" />
 </robot>

File: delicar_description/urdf/robot/delicar_description.urdf.xacro (robot description, xacro)
@@ -4,276 +4,216 @@
     <!-- Constants for robot dimensions -->
     <xacro:property name="PI" value="3.1415926535897931" />
-    <xacro:property name="base_mass" value="50.0" />
-    <xacro:property name="base_width" value="1" />
-    <xacro:property name="base_length" value="1.6" />
-    <xacro:property name="base_height" value="0.4" />
-    <xacro:property name="wheelbase" value="1.2" />
-    <xacro:property name="wheeltrack" value="1.0" />
-    <xacro:property name="wheel_mass" value="5" />
-    <xacro:property name="wheel_len" value="0.1" />
+    <xacro:property name="base_mass" value="40.0" /> <!-- arbitrary value for base mass -->
+    <xacro:property name="base_width" value="1.020" />
+    <xacro:property name="base_length" value="2.062" />
+    <xacro:property name="base_height" value="1.212" />
+    <xacro:property name="wheelbase" value="1.197" />
+    <xacro:property name="wheel_mass" value="1" /> <!-- arbitrary value for wheel mass -->
+    <xacro:property name="wheel_len" value="0.12" />
     <xacro:property name="wheel_radius" value="0.225" />
+    <xacro:property name="wheeltrack" value="1.00" />
     <!-- Base Link -->
     <link name="${prefix}base_link" />
     <!-- Chassis -->
     <link name="${prefix}chassis_link">
-      <visual>
+      <collision>
         <origin xyz="0 0 0" rpy="0 0 0" />
         <geometry>
           <box size="${base_length} ${base_width} ${base_height}" />
         </geometry>
-        <material name="red">
-          <color rgba="1.0 0.2 0.2 1.0" />
+      </collision>
+      <visual>
+        <origin xyz="0 0 0" rpy="0 0 0" />
+        <geometry>
+          <box size="${base_length} ${base_width} ${base_height}" />
+        </geometry>
+        <material name="orange">
         </material>
       </visual>
-      <!-- <collision>
-        <origin xyz="0 0 0" rpy="0 0 0" />
-        <geometry>
-          <box size="${base_length} ${base_width} ${base_height}" />
-        </geometry>
-      </collision> -->
       <inertial>
         <origin xyz="0 0 0" rpy="0 0 0" />
         <mass value="${base_mass}" />
         <inertia
-          ixx="${base_mass / 12.0 * (base_width*base_width + base_height*base_height)}"
-          ixy="0.0"
-          ixz="0.0"
-          iyy="${base_mass / 12.0 * (base_width*base_width + base_height*base_height)}"
-          iyz="0.0"
-          izz="${base_mass / 12.0 * (base_width*base_width + base_height*base_height)}" />
-      </inertial>
-    </link>
-    <!-- Fix color bug in gazebo -->
-    <gazebo reference="${prefix}chassis_link">
-      <visual>
-        <material>
-          <ambient>1.0 0.2 0.2 1.0</ambient>
-          <diffuse>1.0 0.2 0.2 1.0</diffuse>
-          <specular>1.0 1.0 1.0 1.0</specular>
-          <emissive>0.2 0.0 0.0 1.0</emissive>
-        </material>
-      </visual>
-    </gazebo>
-    <!-- Chassis Joint -->
+          ixx="0.000270" ixy="0.0" ixz="0.0"
+          iyy="0.000270" iyz="0.0"
+          izz="0.000426" />
+      </inertial>
+    </link>
     <joint name="${prefix}chassis_joint" type="fixed">
       <parent link="${prefix}base_link" />
       <child link="${prefix}chassis_link" />
-      <origin xyz="0 0 ${wheel_radius + base_height/2}" rpy="0 0 0" />
-    </joint>
-    <!-- Rear wheels -->
+      <origin xyz="0 0 ${base_height/2 + 0.153}" rpy="0 0 0" />
+      <axis xyz="0 0 1" />
+      <dynamics damping="0.2" />
+    </joint>
+    <!-- rear wheels -->
+    <!-- virtual rear wheel -->
+    <link name="${prefix}virtual_rear_wheel">
+      <visual>
+        <origin xyz="0 0 0" rpy="${PI/2} 0 ${PI/2}" />
+        <geometry>
+          <cylinder length="0.01" radius="${wheel_radius}" />
+        </geometry>
+        <material name="invisible" />
+      </visual>
+    </link>
+    <joint name="${prefix}virtual_rear_wheel_joint" type="continuous">
+      <parent link="${prefix}base_link" />
+      <child link="${prefix}virtual_rear_wheel" />
+      <origin xyz="-${wheelbase/2} 0 ${wheel_radius}" rpy="0 0 ${PI/2}" />
+      <axis xyz="1 0 0" />
+      <limit effort="100.0" velocity="100.0" />
+      <dynamics damping="0.2" />
+    </joint>
+    <!-- rear right wheel -->
+    <link name="${prefix}rear_right_wheel">
+      <collision>
+        <origin xyz="0 0 0" rpy="${PI/2} 0 ${PI/2}" />
+        <geometry>
+          <cylinder length="${wheel_len}" radius="${wheel_radius}" />
+        </geometry>
+      </collision>
+      <visual>
+        <origin xyz="0 0 0" rpy="${PI/2} 0 ${PI/2}" />
+        <geometry>
+          <cylinder length="${wheel_len}" radius="${wheel_radius}" />
+        </geometry>
+        <material name="black" />
+      </visual>
+      <inertial>
+        <origin xyz="0 0 0" rpy="${PI/2} 0 ${PI/2}" />
+        <mass value="${wheel_mass}" />
+        <inertia
+          ixx="0.000270" ixy="0.0" ixz="0.0"
+          iyy="0.000270" iyz="0.0"
+          izz="0.000426" />
+      </inertial>
+    </link>
+    <joint name="${prefix}rear_right_wheel_joint" type="continuous">
+      <parent link="${prefix}base_link" />
+      <child link="${prefix}rear_right_wheel" />
+      <origin xyz="-${wheelbase/2} ${base_width/2 - wheel_len/2} ${wheel_radius}" rpy="0 0 ${PI/2}" />
+      <axis xyz="1 0 0" />
+      <limit effort="100.0" velocity="100.0" />
+      <dynamics damping="0.2" />
+      <mimic joint="${prefix}virtual_rear_wheel_joint" multiplier="1.0" offset="0.0" />
+    </joint>
     <!-- rear left wheel -->
     <link name="${prefix}rear_left_wheel">
-      <visual>
-        <origin xyz="0 0 0" rpy="0 0 0" />
-        <geometry>
-          <cylinder length="${wheel_len}" radius="${wheel_radius}" />
-        </geometry>
-        <material name="black">
-          <color rgba="0.0 0.0 0.0 1.0" />
-        </material>
-      </visual>
-      <collision>
-        <origin xyz="0 0 0" rpy="0 0 0" />
-        <geometry>
-          <cylinder length="${wheel_len}" radius="${wheel_radius}" />
-        </geometry>
-      </collision>
-      <inertial>
-        <origin xyz="0 0 0" rpy="0 0 0" />
-        <mass value="${wheel_mass}" />
-        <inertia
-          ixx="${wheel_mass / 12.0 * (3 * wheel_radius*wheel_radius + wheel_len*wheel_len)}"
-          ixy="0.0"
-          ixz="0.0"
-          iyy="${wheel_mass / 12.0 * (3 * wheel_radius*wheel_radius + wheel_len*wheel_len)}"
-          iyz="0.0"
-          izz="${wheel_mass / 2.0 * wheel_radius*wheel_radius}" />
+      <collision>
+        <origin xyz="0 0 0" rpy="${PI/2} 0 ${PI/2}" />
+        <geometry>
+          <cylinder length="${wheel_len}" radius="${wheel_radius}" />
+        </geometry>
+      </collision>
+      <visual>
+        <origin xyz="0 0 0" rpy="${PI/2} 0 ${PI/2}" />
+        <geometry>
+          <cylinder length="${wheel_len}" radius="${wheel_radius}" />
+        </geometry>
+        <material name="black" />
+      </visual>
+      <inertial>
+        <origin xyz="0 0 0" rpy="${PI/2} 0 ${PI/2}" />
+        <mass value="${wheel_mass}" />
+        <inertia
+          ixx="0.000270" ixy="0.0" ixz="0.0"
+          iyy="0.000270" iyz="0.0"
+          izz="0.000426" />
       </inertial>
     </link>
     <joint name="${prefix}rear_left_wheel_joint" type="continuous">
-      <parent link="${prefix}chassis_link" />
+      <parent link="${prefix}base_link" />
       <child link="${prefix}rear_left_wheel" />
-      <origin xyz="-${wheelbase/2} ${wheeltrack/2} -${base_height/2}" rpy="-1.57 0 0" />
-      <axis xyz="0 0 1" />
-      <limit effort="1000.0" velocity="100" />
-    </joint>
-    <gazebo reference="${prefix}rear_left_wheel">
-      <visual>
-        <material>
-          <ambient>0.0 0.0 0.0 1.0</ambient>
-          <diffuse>0.0 0.0 0.0 1.0</diffuse>
-          <specular>0.5 0.5 0.5 1.0</specular>
-          <emissive>0.0 0.0 0.0 1.0</emissive>
-        </material>
-      </visual>
-    </gazebo>
-    <!-- rear right wheel -->
-    <link name="${prefix}rear_right_wheel">
-      <visual>
-        <origin xyz="0 0 0" rpy="0 0 0" />
-        <geometry>
-          <cylinder length="${wheel_len}" radius="${wheel_radius}" />
-        </geometry>
-        <material name="black">
-          <color rgba="0.0 0.0 0.0 1.0" />
-        </material>
-      </visual>
-      <collision>
-        <origin xyz="0 0 0" rpy="0 0 0" />
-        <geometry>
-          <cylinder length="${wheel_len}" radius="${wheel_radius}" />
-        </geometry>
-      </collision>
-      <inertial>
-        <origin xyz="0 0 0" rpy="0 0 0" />
-        <mass value="${wheel_mass}" />
-        <inertia
-          ixx="${wheel_mass / 12.0 * (3 * wheel_radius*wheel_radius + wheel_len*wheel_len)}"
-          ixy="0.0"
-          ixz="0.0"
-          iyy="${wheel_mass / 12.0 * (3 * wheel_radius*wheel_radius + wheel_len*wheel_len)}"
-          iyz="0.0"
-          izz="${wheel_mass / 2.0 * wheel_radius*wheel_radius}" />
-      </inertial>
-    </link>
-    <joint name="${prefix}rear_right_wheel_joint" type="continuous">
-      <parent link="${prefix}chassis_link" />
-      <child link="${prefix}rear_right_wheel" />
-      <origin xyz="-${wheelbase/2} -${wheeltrack/2} -${base_height/2}" rpy="-1.57 0 0" />
-      <axis xyz="0 0 1" />
-      <limit effort="1000.0" velocity="100" />
-    </joint>
-    <gazebo reference="${prefix}rear_right_wheel">
-      <visual>
-        <material>
-          <ambient>0.0 0.0 0.0 1.0</ambient>
-          <diffuse>0.0 0.0 0.0 1.0</diffuse>
-          <specular>0.5 0.5 0.5 1.0</specular>
-          <emissive>0.0 0.0 0.0 1.0</emissive>
-        </material>
-      </visual>
-    </gazebo>
-    <!-- steering links-->
-    <!-- left sterring link-->
-    <link name="${prefix}left_wheel_steering">
-      <inertial>
-        <mass value="0.1" />
-        <inertia ixx="0.001" ixy="0.0" ixz="0.0" iyy="0.001" iyz="0.0" izz="0.001" />
-      </inertial>
-    </link>
-    <!-- left sterring joint-->
-    <joint name="${prefix}left_wheel_steering_joint" type="revolute">
-      <parent link="${prefix}chassis_link" />
-      <child link="${prefix}left_wheel_steering" />
-      <origin xyz="${wheelbase/2} -${wheeltrack/2} -${base_height/2}" rpy="${PI/2} 0 0" />
-      <axis xyz="0 1 0" />
-      <limit effort="1000.0" lower="-1.0471975512" upper="1.0471975512" velocity="30" />
-    </joint>
-    <!-- right sterring link-->
-    <link name="${prefix}right_wheel_steering">
-      <inertial>
-        <mass value="0.1" />
-        <inertia ixx="0.001" ixy="0.0" ixz="0.0" iyy="0.001" iyz="0.0" izz="0.001" />
-      </inertial>
-    </link>
-    <!-- right sterring joint-->
-    <joint name="${prefix}right_wheel_steering_joint" type="revolute">
-      <parent link="${prefix}chassis_link" />
-      <child link="${prefix}right_wheel_steering" />
-      <origin xyz="${wheelbase/2} ${wheeltrack/2} -${base_height/2}" rpy="${PI/2} 0 0" />
-      <axis xyz="0 1 0" />
-      <limit effort="1000.0" lower="-1.0471975512" upper="1.0471975512" velocity="30" />
+      <origin xyz="-${wheelbase/2} -${base_width/2 - wheel_len/2} ${wheel_radius}" rpy="0 0 ${PI/2}" />
+      <axis xyz="1 0 0" />
+      <limit effort="100.0" velocity="100.0" />
+      <dynamics damping="0.2" />
+      <mimic joint="${prefix}virtual_rear_wheel_joint" multiplier="1.0" offset="0.0" />
     </joint>
     <!-- front wheels -->
+    <!-- virtual front wheel -->
+    <link name="${prefix}virtual_front_wheel">
+      <visual>
+        <origin xyz="0 0 0" rpy="${PI/2} 0 ${PI/2}" />
+        <geometry>
+          <cylinder length="0.01" radius="${wheel_radius}" />
+        </geometry>
+        <material name="invisible" />
+      </visual>
+    </link>
+    <joint name="${prefix}virtual_front_wheel_joint" type="revolute">
+      <parent link="${prefix}base_link" />
+      <child link="${prefix}virtual_front_wheel" />
+      <origin xyz="${wheelbase/2} 0 ${wheel_radius}" rpy="0 0 ${PI/2}" />
+      <axis xyz="0 0 1" />
+      <limit lower="-0.4" upper="0.4" effort="100.0" velocity="0.0" />
+      <dynamics damping="0.2" />
+    </joint>
+    <!-- front right wheel -->
+    <link name="${prefix}front_right_wheel">
+      <collision>
+        <origin xyz="0 0 0" rpy="${PI/2} 0 ${PI/2}" />
+        <geometry>
+          <cylinder length="${wheel_len}" radius="${wheel_radius}" />
+        </geometry>
+      </collision>
+      <visual>
+        <origin xyz="0 0 0" rpy="${PI/2} 0 ${PI/2}" />
+        <geometry>
+          <cylinder length="${wheel_len}" radius="${wheel_radius}" />
+        </geometry>
+        <material name="black" />
+      </visual>
+      <inertial>
+        <origin xyz="0 0 0" rpy="${PI/2} 0 ${PI/2}" />
+        <mass value="${wheel_mass}" />
+        <inertia
+          ixx="0.000270" ixy="0.0" ixz="0.0"
+          iyy="0.000270" iyz="0.0"
+          izz="0.000426" />
+      </inertial>
+    </link>
+    <joint name="${prefix}front_right_wheel_joint" type="revolute">
+      <parent link="${prefix}base_link" />
+      <child link="${prefix}front_right_wheel" />
+      <origin xyz="${wheelbase/2} ${base_width/2 - wheel_len/2} ${wheel_radius}" rpy="0 0 ${PI/2}" />
+      <axis xyz="0 0 1" />
+      <limit lower="-0.4" upper="0.4" effort="100.0" velocity="0.0" />
+      <dynamics damping="0.2" />
+      <mimic joint="${prefix}virtual_front_wheel_joint" multiplier="1.0" offset="0.0" />
+    </joint>
     <!-- front left steering -->
     <link name="${prefix}front_left_wheel">
       <collision>
-        <origin xyz="0 0 0" rpy="0 0 0" />
-        <geometry>
-          <cylinder length="${wheel_len}" radius="${wheel_radius}" />
-        </geometry>
-      </collision>
-      <visual>
-        <origin xyz="0 0 0" rpy="0 0 0" />
-        <geometry>
-          <cylinder length="${wheel_len}" radius="${wheel_radius}" />
-        </geometry>
-        <material name="black" />
-      </visual>
-      <inertial>
-        <origin xyz="0 0 0" rpy="0 0 0" />
-        <mass value="${wheel_mass}" />
-        <inertia
-          ixx="${wheel_mass / 12.0 * (3 * wheel_radius*wheel_radius + wheel_len*wheel_len)}"
-          ixy="0.0"
-          ixz="0.0"
-          iyy="${wheel_mass / 12.0 * (3 * wheel_radius*wheel_radius + wheel_len*wheel_len)}"
-          iyz="0.0"
-          izz="${wheel_mass / 2.0 * wheel_radius*wheel_radius}" />
-      </inertial>
-    </link>
-    <joint name="${prefix}front_left_wheel_joint" type="continuous">
-      <parent link="${prefix}left_wheel_steering" />
+        <origin xyz="0 0 0" rpy="${PI/2} 0 ${PI/2}" />
+        <geometry>
+          <cylinder length="${wheel_len}" radius="${wheel_radius}" />
+        </geometry>
+      </collision>
+      <visual>
+        <origin xyz="0 0 0" rpy="${PI/2} 0 ${PI/2}" />
+        <geometry>
+          <cylinder length="${wheel_len}" radius="${wheel_radius}" />
+        </geometry>
+        <material name="black" />
+      </visual>
+      <inertial>
+        <origin xyz="0 0 0" rpy="${PI/2} 0 ${PI/2}" />
+        <mass value="${wheel_mass}" />
+        <inertia
+          ixx="0.000270" ixy="0.0" ixz="0.0"
+          iyy="0.000270" iyz="0.0"
+          izz="0.000426" />
+      </inertial>
+    </link>
+    <joint name="${prefix}front_left_wheel_joint" type="revolute">
+      <parent link="${prefix}base_link" />
       <child link="${prefix}front_left_wheel" />
-      <origin xyz="0 0 0" rpy="0 0 0" />
-      <axis xyz="0 0 1" />
-    </joint>
-    <!-- front right wheel -->
-    <link name="${prefix}front_right_wheel">
-      <collision>
-        <origin xyz="0 0 0" rpy="0 0 0" />
-        <geometry>
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
File: delicar_description/urdf/sensors/imu.urdf.xacro (robot description, xacro)
@@ -5,5 +5,5 @@
       <parent link="${prefix}base_link" />
       <child link="${prefix}imu_link" />
-      <origin xyz="0 0 0.425" rpy="0 0 0" />
+      <origin xyz="0.93 0 1.475" rpy="0 0.261 0" />
     </joint>
     <gazebo reference="${prefix}imu_link">
