Commit message: Change lidar_3d urdf to rslidar urdf

File: delicar_description/urdf/delicar.urdf.xacro (robot description, xacro)
@@ -8,5 +8,5 @@
   <!-- <xacro:include filename="$(find delicar_description)/urdf/sensors/depth_camera.urdf.xacro" /> -->
   <xacro:include filename="$(find delicar_description)/urdf/sensors/imu.urdf.xacro" />
-  <xacro:include filename="$(find delicar_description)/urdf/sensors/lidar_3d.urdf.xacro" />
+  <xacro:include filename="$(find delicar_description)/urdf/sensors/rslidar.urdf.xacro" />
   <xacro:include filename="$(find delicar_description)/urdf/controllers/delicar_controllers.xacro" />
   <!-- Import delicar description -->
@@ -17,5 +17,5 @@
   <!-- <xacro:imu prefix="$(arg prefix)"/> -->
   <!-- Import 3d lidar -->
-  <xacro:lidar_3d
+  <xacro:rslidar
     prefix="$(arg prefix)"
     frame_id="rslidar"

File: delicar_description/urdf/sensors/rslidar.urdf.xacro (robot description, xacro)
@@ -1,5 +1,5 @@
 <robot xmlns:xacro="http://ros.org/wiki/xacro">
   <xacro:property name="M_PI" value="3.1415926535897931" />
-  <xacro:macro name="lidar_3d" params="prefix frame_id">
+  <xacro:macro name="rslidar" params="prefix frame_id">
     <link name="${frame_id}">
       <visual>
@@ -29,5 +29,5 @@
       <parent link="${prefix}base_link" />
       <child link="${frame_id}" />
-      <origin xyz="0.93 0 1.535" rpy="0 0.261 0" />
+      <origin xyz="0.93 0 1.4" rpy="0 0 0" />
     </joint>
   </xacro:macro>
